Commit message: Update dg5f_right.xacro

File: dg_description/urdf/dg5f_right.xacro (robot description, xacro)
@@ -130,5 +130,5 @@
     <child link="rl_dg_1_2" />
     <axis xyz="0 0 1" />
-    <limit lower="-3.141592653589793" upper="0.01" effort="7.5" velocity="3.141592653589793"/>
+    <limit lower="-3.141592653589793" upper="0.0" effort="7.5" velocity="3.141592653589793"/>
   </joint>
   <link name="rl_dg_1_3">
@@ -156,5 +156,5 @@
     <child link="rl_dg_1_3" />
     <axis xyz="1 0 0" />
-    <limit lower="-0.001" upper="1.5707963267948966" effort="7.5" velocity="3.141592653589793"/>
+    <limit lower="-1.5707963267948966" upper="1.5707963267948966" effort="7.5" velocity="3.141592653589793"/>
   </joint>
   <link name="rl_dg_1_4">
@@ -182,5 +182,5 @@
     <child link="rl_dg_1_4" />
     <axis xyz="1 0 0" />
-    <limit lower="-0.001" upper="1.5707963267948966" effort="7.5" velocity="3.141592653589793"/>
+    <limit lower="-1.5707963267948966" upper="1.5707963267948966" effort="7.5" velocity="3.141592653589793"/>
   </joint>
   <link name="rl_dg_1_tip">
@@ -284,5 +284,5 @@
     <child link="rl_dg_2_3" />
     <axis xyz="0 1 0" />
-    <limit lower="-0.01" upper="1.5707963267948966" effort="7.5" velocity="3.141592653589793"/>
+    <limit lower="-1.5707963267948966" upper="1.5707963267948966" effort="7.5" velocity="3.141592653589793"/>
   </joint>
   <link name="rl_dg_2_4">
@@ -310,5 +310,5 @@
     <child link="rl_dg_2_4" />
     <axis xyz="0 1 0" />
-    <limit lower="-0.01" upper="1.5707963267948966" effort="7.5" velocity="3.141592653589793"/>
+    <limit lower="-1.5707963267948966" upper="1.5707963267948966" effort="7.5" velocity="3.141592653589793"/>
   </joint>
   <link name="rl_dg_2_tip">
@@ -386,5 +386,5 @@
     <child link="rl_dg_3_2" />
     <axis xyz="0 1 0" />
-    <limit lower="-0.01" upper="1.9547687622336491" effort="7.5" velocity="3.141592653589793"/>
+    <limit lower="-0.0" upper="1.9547687622336491" effort="7.5" velocity="3.141592653589793"/>
   </joint>
   <link name="rl_dg_3_3">
@@ -412,5 +412,5 @@
     <child link="rl_dg_3_3" />
     <axis xyz="0 1 0" />
-    <limit lower="-0.01" upper="1.5707963267948966" effort="7.5" velocity="3.141592653589793"/>
+    <limit lower="-1.5707963267948966" upper="1.5707963267948966" effort="7.5" velocity="3.141592653589793"/>
   </joint>
   <link name="rl_dg_3_4">
@@ -438,5 +438,5 @@
     <child link="rl_dg_3_4" />
     <axis xyz="0 1 0" />
-    <limit lower="-0.01" upper="1.5707963267948966" effort="7.5" velocity="3.141592653589793"/>
+    <limit lower="-1.5707963267948966" upper="1.5707963267948966" effort="7.5" velocity="3.141592653589793"/>
   </joint>
   <link name="rl_dg_3_tip">
@@ -514,5 +514,5 @@
     <child link="rl_dg_4_2" />
     <axis xyz="0 1 0" />
-    <limit lower="-0.01" upper="1.9024088846738192" effort="7.5" velocity="3.141592653589793"/>
+    <limit lower="-0.0" upper="1.9024088846738192" effort="7.5" velocity="3.141592653589793"/>
   </joint>
   <link name="rl_dg_4_3">
@@ -540,5 +540,5 @@
     <child link="rl_dg_4_3" />
     <axis xyz="0 1 0" />
-    <limit lower="-0.01" upper="1.5707963267948966" effort="7.5" velocity="3.141592653589793"/>
+    <limit lower="-1.5707963267948966" upper="1.5707963267948966" effort="7.5" velocity="3.141592653589793"/>
   </joint>
   <link name="rl_dg_4_4">
@@ -566,5 +566,5 @@
     <child link="rl_dg_4_4" />
     <axis xyz="0 1 0" />
-    <limit lower="-0.01" upper="1.5707963267948966" effort="7.5" velocity="3.141592653589793"/>
+    <limit lower="-1.5707963267948966" upper="1.5707963267948966" effort="7.5" velocity="3.141592653589793"/>
   </joint>
   <link name="rl_dg_4_tip">
@@ -668,5 +668,5 @@
     <child link="rl_dg_5_3" />
     <axis xyz="0 1 0" />
-    <limit lower="-0.01" upper="1.5707963267948966" effort="7.5" velocity="3.141592653589793"/>
+    <limit lower="-1.5707963267948966" upper="1.5707963267948966" effort="7.5" velocity="3.141592653589793"/>
   </joint>
   <link name="rl_dg_5_4">
@@ -694,5 +694,5 @@
     <child link="rl_dg_5_4" />
     <axis xyz="0 1 0" />
-    <limit lower="-0.01" upper="1.5707963267948966" effort="7.5" velocity="3.141592653589793"/>
+    <limit lower="-1.5707963267948966" upper="1.5707963267948966" effort="7.5" velocity="3.141592653589793"/>
   </joint>
   <link name="rl_dg_5_tip">
