Commit message: update description files.

File: dg_description/urdf/dg5f_left.urdf (robot description, URDF)
Before this commit: robot dg5f_left, 28 links, 27 joints
Links:
- link ll_dg_1_1: geometry collision mesh filename=package://meshes/dg5f_left/collision/ll_dg_1_1_c.STL; visual mesh filename=package://meshes/dg5f_left/visual/ll_dg_1_1.dae
- link ll_dg_1_2: geometry collision mesh filename=package://meshes/dg5f_left/collision/ll_dg_1_2_c.STL; visual mesh filename=package://meshes/dg5f_left/visual/ll_dg_1_2.dae
- link ll_dg_1_3: geometry collision mesh filename=package://meshes/dg5f_left/collision/ll_dg_1_3_c.STL; visual mesh filename=package://meshes/dg5f_left/visual/ll_dg_1_3.dae
- link ll_dg_1_4: geometry collision mesh filename=package://meshes/dg5f_left/collision/ll_dg_1_4_c.STL; visual mesh filename=package://meshes/dg5f_left/visual/ll_dg_1_4.dae
- link ll_dg_1_tip: geometry collision mesh filename=package://meshes/dg5f_left/collision/ll_dg_1_tip_c.STL; visual mesh filename=package://meshes/dg5f_left/visual/ll_dg_1_tip.dae
- link ll_dg_2_1: geometry collision mesh filename=package://meshes/dg5f_left/collision/ll_dg_2_1_c.STL; visual mesh filename=package://meshes/dg5f_left/visual/ll_dg_2_1.dae
- link ll_dg_2_2: geometry collision mesh filename=package://meshes/dg5f_left/collision/ll_dg_2_2_c.STL; visual mesh filename=package://meshes/dg5f_left/visual/ll_dg_2_2.dae
- link ll_dg_2_3: geometry collision mesh filename=package://meshes/dg5f_left/collision/ll_dg_2_3_c.STL; visual mesh filename=package://meshes/dg5f_left/visual/ll_dg_2_3.dae
- link ll_dg_2_4: geometry collision mesh filename=package://meshes/dg5f_left/collision/ll_dg_2_4_c.STL; visual mesh filename=package://meshes/dg5f_left/visual/ll_dg_2_4.dae
- link ll_dg_2_tip: geometry collision mesh filename=package://meshes/dg5f_left/collision/ll_dg_2_tip_c.STL; visual mesh filename=package://meshes/dg5f_left/visual/ll_dg_2_tip.dae
- link ll_dg_3_1: geometry collision mesh filename=package://meshes/dg5f_left/collision/ll_dg_3_1_c.STL; visual mesh filename=package://meshes/dg5f_left/visual/ll_dg_3_1.dae
- link ll_dg_3_2: geometry collision mesh filename=package://meshes/dg5f_left/collision/ll_dg_3_2_c.STL; visual mesh filename=package://meshes/dg5f_left/visual/ll_dg_3_2.dae
- link ll_dg_3_3: geometry collision mesh filename=package://meshes/dg5f_left/collision/ll_dg_3_3_c.STL; visual mesh filename=package://meshes/dg5f_left/visual/ll_dg_3_3.dae
- link ll_dg_3_4: geometry collision mesh filename=package://meshes/dg5f_left/collision/ll_dg_3_4_c.STL; visual mesh filename=package://meshes/dg5f_left/visual/ll_dg_3_4.dae
- link ll_dg_3_tip: geometry collision mesh filename=package://meshes/dg5f_left/collision/ll_dg_3_tip_c.STL; visual mesh filename=package://meshes/dg5f_left/visual/ll_dg_3_tip.dae
- link ll_dg_4_1: geometry collision mesh filename=package://meshes/dg5f_left/collision/ll_dg_4_1_c.STL; visual mesh filename=package://meshes/dg5f_left/visual/ll_dg_4_1.dae
- link ll_dg_4_2: geometry collision mesh filename=package://meshes/dg5f_left/collision/ll_dg_4_2_c.STL; visual mesh filename=package://meshes/dg5f_left/visual/ll_dg_4_2.dae
- link ll_dg_4_3: geometry collision mesh filename=package://meshes/dg5f_left/collision/ll_dg_4_3_c.STL; visual mesh filename=package://meshes/dg5f_left/visual/ll_dg_4_3.dae
- link ll_dg_4_4: geometry collision mesh filename=package://meshes/dg5f_left/collision/ll_dg_4_4_c.STL; visual mesh filename=package://meshes/dg5f_left/visual/ll_dg_4_4.dae
- link ll_dg_4_tip: geometry collision mesh filename=package://meshes/dg5f_left/collision/ll_dg_4_tip_c.STL; visual mesh filename=package://meshes/dg5f_left/visual/ll_dg_4_tip.dae
- link ll_dg_5_1: geometry collision mesh filename=package://meshes/dg5f_left/collision/ll_dg_5_1_c.STL; visual mesh filename=package://meshes/dg5f_left/visual/ll_dg_5_1.dae
- link ll_dg_5_2: geometry collision mesh filename=package://meshes/dg5f_left/collision/ll_dg_5_2_c.STL; visual mesh filename=package://meshes/dg5f_left/visual/ll_dg_5_2.dae
- link ll_dg_5_3: geometry collision mesh filename=package://meshes/dg5f_left/collision/ll_dg_5_3_c.STL; visual mesh filename=package://meshes/dg5f_left/visual/ll_dg_5_3.dae
- link ll_dg_5_4: geometry collision mesh filename=package://meshes/dg5f_left/collision/ll_dg_5_4_c.STL; visual mesh filename=package://meshes/dg5f_left/visual/ll_dg_5_4.dae
- link ll_dg_5_tip: geometry collision mesh filename=package://meshes/dg5f_left/collision/ll_dg_5_tip_c.STL; visual mesh filename=package://meshes/dg5f_left/visual/ll_dg_5_tip.dae
- link ll_dg_base: geometry collision mesh filename=package://meshes/dg5f_left/collision/ll_dg_base_c.STL; visual mesh filename=package://meshes/dg5f_left/visual/ll_dg_base.dae
- link ll_dg_mount: geometry collision mesh filename=package://meshes/dg5f_left/collision/ll_dg_mount_c.STL; visual mesh filename=package://meshes/dg5f_left/visual/ll_dg_mount.dae
- link ll_dg_palm: geometry collision mesh filename=package://meshes/dg5f_left/collision/ll_dg_palm_c.STL; visual mesh filename=package://meshes/dg5f_left/visual/ll_dg_palm.dae
Joints:
- joint lj_dg_1_3: limit lower=-1.5707963267948966 upper=0.0 effort=7.5 velocity=3.141592653589793 -> lower=-1.5707963267948966 upper=1.5707963267948966 effort=7.5 velocity=3.141592653589793
- joint lj_dg_1_4: limit lower=-1.5707963267948966 upper=0.0 effort=7.5 velocity=3.141592653589793 -> lower=-1.5707963267948966 upper=1.5707963267948966 effort=7.5 velocity=3.141592653589793
- joint lj_dg_2_3: limit lower=0.0 upper=1.5707963267948966 effort=7.5 velocity=3.141592653589793 -> lower=-1.5707963267948966 upper=1.5707963267948966 effort=7.5 velocity=3.141592653589793
- joint lj_dg_2_4: limit lower=0.0 upper=1.5707963267948966 effort=7.5 velocity=3.141592653589793 -> lower=-1.5707963267948966 upper=1.5707963267948966 effort=7.5 velocity=3.141592653589793
- joint lj_dg_3_3: limit lower=0.0 upper=1.5707963267948966 effort=7.5 velocity=3.141592653589793 -> lower=-1.5707963267948966 upper=1.5707963267948966 effort=7.5 velocity=3.141592653589793
- joint lj_dg_3_4: limit lower=0.0 upper=1.5707963267948966 effort=7.5 velocity=3.141592653589793 -> lower=-1.5707963267948966 upper=1.5707963267948966 effort=7.5 velocity=3.141592653589793
- joint lj_dg_4_3: limit lower=0.0 upper=1.5707963267948966 effort=7.5 velocity=3.141592653589793 -> lower=-1.5707963267948966 upper=1.5707963267948966 effort=7.5 velocity=3.141592653589793
- joint lj_dg_4_4: limit lower=0.0 upper=1.5707963267948966 effort=7.5 velocity=3.141592653589793 -> lower=-1.5707963267948966 upper=1.5707963267948966 effort=7.5 velocity=3.141592653589793
- joint lj_dg_5_3: limit lower=0.0 upper=1.5707963267948966 effort=7.5 velocity=3.141592653589793 -> lower=-1.5707963267948966 upper=1.5707963267948966 effort=7.5 velocity=3.141592653589793
- joint lj_dg_5_4: limit lower=0.0 upper=1.5707963267948966 effort=7.5 velocity=3.141592653589793 -> lower=-1.5707963267948966 upper=1.5707963267948966 effort=7.5 velocity=3.141592653589793

File: dg_description/urdf/dg5f_left.xacro (robot description, xacro)
@@ -284,5 +284,5 @@
     <child link="ll_dg_2_3" />
     <axis xyz="0 1 0" />
-    <limit lower="-0.01" upper="1.5707963267948966" effort="7.5" velocity="3.141592653589793"/>
+    <limit lower="-1.5707963267948966" upper="1.5707963267948966" effort="7.5" velocity="3.141592653589793"/>
   </joint>
   <link name="ll_dg_2_4">
@@ -310,5 +310,5 @@
     <child link="ll_dg_2_4" />
     <axis xyz="0 1 0" />
-    <limit lower="-0.01" upper="1.5707963267948966" effort="7.5" velocity="3.141592653589793"/>
+    <limit lower="-1.5707963267948966" upper="1.5707963267948966" effort="7.5" velocity="3.141592653589793"/>
   </joint>
   <link name="ll_dg_2_tip">

File: dg_description/urdf/dg5f_right.urdf (robot description, URDF)
Before this commit: robot dg5f_right, 28 links, 27 joints
Links:
- link rl_dg_1_1: geometry collision mesh filename=package://meshes/dg5f_right/collision/rl_dg_1_1_c.STL; visual mesh filename=package://meshes/dg5f_right/visual/rl_dg_1_1.dae
- link rl_dg_1_2: geometry collision mesh filename=package://meshes/dg5f_right/collision/rl_dg_1_2_c.STL; visual mesh filename=package://meshes/dg5f_right/visual/rl_dg_1_2.dae
- link rl_dg_1_3: geometry collision mesh filename=package://meshes/dg5f_right/collision/rl_dg_1_3_c.STL; visual mesh filename=package://meshes/dg5f_right/visual/rl_dg_1_3.dae
- link rl_dg_1_4: geometry collision mesh filename=package://meshes/dg5f_right/collision/rl_dg_1_4_c.STL; visual mesh filename=package://meshes/dg5f_right/visual/rl_dg_1_4.dae
- link rl_dg_1_tip: geometry collision mesh filename=package://meshes/dg5f_right/collision/rl_dg_1_tip_c.STL; visual mesh filename=package://meshes/dg5f_right/visual/rl_dg_1_tip.dae
- link rl_dg_2_1: geometry collision mesh filename=package://meshes/dg5f_right/collision/rl_dg_2_1_c.STL; visual mesh filename=package://meshes/dg5f_right/visual/rl_dg_2_1.dae
- link rl_dg_2_2: geometry collision mesh filename=package://meshes/dg5f_right/collision/rl_dg_2_2_c.STL; visual mesh filename=package://meshes/dg5f_right/visual/rl_dg_2_2.dae
- link rl_dg_2_3: geometry collision mesh filename=package://meshes/dg5f_right/collision/rl_dg_2_3_c.STL; visual mesh filename=package://meshes/dg5f_right/visual/rl_dg_2_3.dae
- link rl_dg_2_4: geometry collision mesh filename=package://meshes/dg5f_right/collision/rl_dg_2_4_c.STL; visual mesh filename=package://meshes/dg5f_right/visual/rl_dg_2_4.dae
- link rl_dg_2_tip: geometry collision mesh filename=package://meshes/dg5f_right/collision/rl_dg_2_tip_c.STL; visual mesh filename=package://meshes/dg5f_right/visual/rl_dg_2_tip.dae
- link rl_dg_3_1: geometry collision mesh filename=package://meshes/dg5f_right/collision/rl_dg_3_1_c.STL; visual mesh filename=package://meshes/dg5f_right/visual/rl_dg_3_1.dae
- link rl_dg_3_2: geometry collision mesh filename=package://meshes/dg5f_right/collision/rl_dg_3_2_c.STL; visual mesh filename=package://meshes/dg5f_right/visual/rl_dg_3_2.dae
- link rl_dg_3_3: geometry collision mesh filename=package://meshes/dg5f_right/collision/rl_dg_3_3_c.STL; visual mesh filename=package://meshes/dg5f_right/visual/rl_dg_3_3.dae
- link rl_dg_3_4: geometry collision mesh filename=package://meshes/dg5f_right/collision/rl_dg_3_4_c.STL; visual mesh filename=package://meshes/dg5f_right/visual/rl_dg_3_4.dae
- link rl_dg_3_tip: geometry collision mesh filename=package://meshes/dg5f_right/collision/rl_dg_3_tip_c.STL; visual mesh filename=package://meshes/dg5f_right/visual/rl_dg_3_tip.dae
- link rl_dg_4_1: geometry collision mesh filename=package://meshes/dg5f_right/collision/rl_dg_4_1_c.STL; visual mesh filename=package://meshes/dg5f_right/visual/rl_dg_4_1.dae
- link rl_dg_4_2: geometry collision mesh filename=package://meshes/dg5f_right/collision/rl_dg_4_2_c.STL; visual mesh filename=package://meshes/dg5f_right/visual/rl_dg_4_2.dae
- link rl_dg_4_3: geometry collision mesh filename=package://meshes/dg5f_right/collision/rl_dg_4_3_c.STL; visual mesh filename=package://meshes/dg5f_right/visual/rl_dg_4_3.dae
- link rl_dg_4_4: geometry collision mesh filename=package://meshes/dg5f_right/collision/rl_dg_4_4_c.STL; visual mesh filename=package://meshes/dg5f_right/visual/rl_dg_4_4.dae
- link rl_dg_4_tip: geometry collision mesh filename=package://meshes/dg5f_right/collision/rl_dg_4_tip_c.STL; visual mesh filename=package://meshes/dg5f_right/visual/rl_dg_4_tip.dae
- link rl_dg_5_1: geometry collision mesh filename=package://meshes/dg5f_right/collision/rl_dg_5_1_c.STL; visual mesh filename=package://meshes/dg5f_right/visual/rl_dg_5_1.dae
- link rl_dg_5_2: geometry collision mesh filename=package://meshes/dg5f_right/collision/rl_dg_5_2_c.STL; visual mesh filename=package://meshes/dg5f_right/visual/rl_dg_5_2.dae
- link rl_dg_5_3: geometry collision mesh filename=package://meshes/dg5f_right/collision/rl_dg_5_3_c.STL; visual mesh filename=package://meshes/dg5f_right/visual/rl_dg_5_3.dae
- link rl_dg_5_4: geometry collision mesh filename=package://meshes/dg5f_right/collision/rl_dg_5_4_c.STL; visual mesh filename=package://meshes/dg5f_right/visual/rl_dg_5_4.dae
- link rl_dg_5_tip: geometry collision mesh filename=package://meshes/dg5f_right/collision/rl_dg_5_tip_c.STL; visual mesh filename=package://meshes/dg5f_right/visual/rl_dg_5_tip.dae
- link rl_dg_base: geometry collision mesh filename=package://meshes/dg5f_right/collision/rl_dg_base_c.STL; visual mesh filename=package://meshes/dg5f_right/visual/rl_dg_base.dae
- link rl_dg_mount: geometry collision mesh filename=package://meshes/dg5f_right/collision/rl_dg_mount_c.STL; visual mesh filename=package://meshes/dg5f_right/visual/rl_dg_mount.dae
- link rl_dg_palm: geometry collision mesh filename=package://meshes/dg5f_right/collision/rl_dg_palm_c.STL; visual mesh filename=package://meshes/dg5f_right/visual/rl_dg_palm.dae
Joints:
- joint rj_dg_1_3: limit lower=0.0 upper=1.5707963267948966 effort=7.5 velocity=3.141592653589793 -> lower=-1.5707963267948966 upper=1.5707963267948966 effort=7.5 velocity=3.141592653589793
- joint rj_dg_1_4: limit lower=0.0 upper=1.5707963267948966 effort=7.5 velocity=3.141592653589793 -> lower=-1.5707963267948966 upper=1.5707963267948966 effort=7.5 velocity=3.141592653589793
- joint rj_dg_2_3: limit lower=0.0 upper=1.5707963267948966 effort=7.5 velocity=3.141592653589793 -> lower=-1.5707963267948966 upper=1.5707963267948966 effort=7.5 velocity=3.141592653589793
- joint rj_dg_2_4: limit lower=0.0 upper=1.5707963267948966 effort=7.5 velocity=3.141592653589793 -> lower=-1.5707963267948966 upper=1.5707963267948966 effort=7.5 velocity=3.141592653589793
- joint rj_dg_3_3: limit lower=0.0 upper=1.5707963267948966 effort=7.5 velocity=3.141592653589793 -> lower=-1.5707963267948966 upper=1.5707963267948966 effort=7.5 velocity=3.141592653589793
- joint rj_dg_3_4: limit lower=0.0 upper=1.5707963267948966 effort=7.5 velocity=3.141592653589793 -> lower=-1.5707963267948966 upper=1.5707963267948966 effort=7.5 velocity=3.141592653589793
- joint rj_dg_4_3: limit lower=0.0 upper=1.5707963267948966 effort=7.5 velocity=3.141592653589793 -> lower=-1.5707963267948966 upper=1.5707963267948966 effort=7.5 velocity=3.141592653589793
- joint rj_dg_4_4: limit lower=0.0 upper=1.5707963267948966 effort=7.5 velocity=3.141592653589793 -> lower=-1.5707963267948966 upper=1.5707963267948966 effort=7.5 velocity=3.141592653589793
- joint rj_dg_5_3: limit lower=0.0 upper=1.5707963267948966 effort=7.5 velocity=3.141592653589793 -> lower=-1.5707963267948966 upper=1.5707963267948966 effort=7.5 velocity=3.141592653589793
- joint rj_dg_5_4: limit lower=0.0 upper=1.5707963267948966 effort=7.5 velocity=3.141592653589793 -> lower=-1.5707963267948966 upper=1.5707963267948966 effort=7.5 velocity=3.141592653589793
