Commit message: update dg3fm model.

File: dg_description/urdf/dg3f_m.urdf (robot description, URDF)
Before this commit: robot dg3f_m, 16 links, 15 joints
Links:
- removed link l_1_1
- removed link l_1_2
- removed link l_1_3
- removed link l_1_4
- removed link l_1_tip
- removed link l_2_1
- removed link l_2_2
- removed link l_2_3
- removed link l_2_4
- removed link l_2_tip
- removed link l_3_1
- removed link l_3_2
- removed link l_3_3
- removed link l_3_4
- removed link l_3_tip
- removed link l_base
- added link l_dg_1_1, mass 0.0493; collision mesh filename=package://dg_description/meshes/dg3f_m/collision/l_1_1_c.STL; visual mesh filename=package://dg_description/meshes/dg3f_m/visual/l_1_1.dae
- added link l_dg_1_2, mass 0.0191; collision mesh filename=package://dg_description/meshes/dg3f_m/collision/l_1_2_c.STL; visual mesh filename=package://dg_description/meshes/dg3f_m/visual/l_1_2.dae
- added link l_dg_1_3, mass 0.04535; collision mesh filename=package://dg_description/meshes/dg3f_m/collision/l_1_3_c.STL; visual mesh filename=package://dg_description/meshes/dg3f_m/visual/l_1_3.dae
- added link l_dg_1_4, mass 0.0408; collision mesh filename=package://dg_description/meshes/dg3f_m/collision/l_1_4_c.STL; visual mesh filename=package://dg_description/meshes/dg3f_m/visual/l_1_4.dae
- added link l_dg_1_tip, mass 0.0172; collision mesh filename=package://dg_description/meshes/dg3f_m/collision/l_1_tip_c.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; visual mesh filename=package://dg_description/meshes/dg3f_m/visual/l_1_tip.dae
- added link l_dg_2_1, mass 0.0493; collision mesh filename=package://dg_description/meshes/dg3f_m/collision/l_23_1_c.S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; visual mesh filename=package://dg_description/meshes/dg3f_m/visual/l_23_1.dae
- added link l_dg_2_2, mass 0.0191; collision mesh filename=package://dg_description/meshes/dg3f_m/collision/l_23_2_c.S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; visual mesh filename=package://dg_description/meshes/dg3f_m/visual/l_23_2.dae
- added link l_dg_2_3, mass 0.04535; collision mesh filename=package://dg_description/meshes/dg3f_m/collision/l_23_3_c.S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; visual mesh filename=package://dg_description/meshes/dg3f_m/visual/l_23_3.dae
- added link l_dg_2_4, mass 0.0408; collision mesh filename=package://dg_description/meshes/dg3f_m/collision/l_23_4_c.S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; visual mesh filename=package://dg_description/meshes/dg3f_m/visual/l_23_4.dae
- added link l_dg_2_tip, mass 0.0172; collision mesh filename=package://dg_description/meshes/dg3f_m/collision/l_23_tip_c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; visual mesh filename=package://dg_description/meshes/dg3f_m/visual/l_23_tip.dae
- added link l_dg_3_1, mass 0.0493; collision mesh filename=package://dg_description/meshes/dg3f_m/collision/l_23_1_c.S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; visual mesh filename=package://dg_description/meshes/dg3f_m/visual/l_23_1.dae
- added link l_dg_3_2, mass 0.0191; collision mesh filename=package://dg_description/meshes/dg3f_m/collision/l_23_2_c.S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; visual mesh filename=package://dg_description/meshes/dg3f_m/visual/l_23_2.dae
- added link l_dg_3_3, mass 0.04535; collision mesh filename=package://dg_description/meshes/dg3f_m/collision/l_23_3_c.S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; visual mesh filename=package://dg_description/meshes/dg3f_m/visual/l_23_3.dae
- added link l_dg_3_4, mass 0.0408; collision mesh filename=package://dg_description/meshes/dg3f_m/collision/l_23_4_c.S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; visual mesh filename=package://dg_description/meshes/dg3f_m/visual/l_23_4.dae
- added link l_dg_3_tip, mass 0.0172; collision mesh filename=package://dg_description/meshes/dg3f_m/collision/l_23_tip_c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; visual mesh filename=package://dg_description/meshes/dg3f_m/visual/l_23_tip.dae
- added link l_dg_base, mass 0.451; collision mesh filename=package://dg_description/meshes/dg3f_m/collision/l_dg_base_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; visual mesh filename=package://dg_description/meshes/dg3f_m/visual/l_dg_base.dae
- added link l_dg_mount, mass 0.035; collision mesh filename=package://dg_description/meshes/dg3f_m/collision/l_dg_mount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; visual mesh filename=package://dg_description/meshes/dg3f_m/visual/l_dg_mount.dae
Joints:
- removed joint j_1_1
- removed joint j_1_2
- removed joint j_1_3
- removed joint j_1_4
- removed joint j_1_tip
- removed joint j_2_1
- removed joint j_2_2
- removed joint j_2_3
- removed joint j_2_4
- removed joint j_2_tip
- removed joint j_3_1
- removed joint j_3_2
- removed joint j_3_3
- removed joint j_3_4
- removed joint j_3_tip
- added joint j_dg_1_1: type revolute, parent l_dg_base, child l_dg_1_1, origin xyz=0.026558 0 0.0712 rpy=0 0 0, axis 0 0 1, limit lower=-1.5707963267948966 upper=1.5707963267948966 effort=7.644 velocity=3.141592653589793
- added joint j_dg_1_2: type revolute, parent l_dg_1_1, child l_dg_1_2, origin xyz=0 0 0.0405 rpy=0 0 0, axis 1 0 0, limit lower=-1.5707963267948966 upper=1.5707963267948966 effort=7.644 velocity=3.141592653589793
- added joint j_dg_1_3: type revolute, parent l_dg_1_2, child l_dg_1_3, origin xyz=0.0242 0 0.029 rpy=0 0 0, axis 0 -1 0, limit lower=-0.0 upper=2.8099800957108707 effort=7.644 velocity=3.141592653589793
- added joint j_dg_1_4: type revolute, parent l_dg_1_3, child l_dg_1_4, origin xyz=0.0434 0 0 rpy=0 0 0, axis 0 -1 0, limit lower=-1.5707963267948966 upper=1.8675022996339325 effort=7.644 velocity=3.141592653589793
- added joint j_dg_1_tip: type fixed, parent l_dg_1_4, child l_dg_1_tip, origin xyz=0.0313 0 0 rpy=0 0 0
- added joint j_dg_2_1: type revolute, parent l_dg_base, child l_dg_2_1, origin xyz=-0.013279 0.023 0.0712 rpy=0 0 0, axis 0 0 1, limit lower=-2.129301687433082 upper=1.5707963267948966 effort=7.644 velocity=3.141592653589793
- added joint j_dg_2_2: type revolute, parent l_dg_2_1, child l_dg_2_2, origin xyz=0 0 0.0405 rpy=0 0 0, axis -1 0 0, limit lower=-1.5707963267948966 upper=1.5707963267948966 effort=7.644 velocity=3.141592653589793
- added joint j_dg_2_3: type revolute, parent l_dg_2_2, child l_dg_2_3, origin xyz=-0.0242 0 0.029 rpy=0 0 0, axis 0 1 0, limit lower=-0.0 upper=2.8099800957108707 effort=7.644 velocity=3.141592653589793
- added joint j_dg_2_4: type revolute, parent l_dg_2_3, child l_dg_2_4, origin xyz=-0.0434 0 0 rpy=0 0 0, axis 0 1 0, limit lower=-1.5707963267948966 upper=1.8675022996339325 effort=7.644 velocity=3.141592653589793
- added joint j_dg_2_tip: type fixed, parent l_dg_2_4, child l_dg_2_tip, origin xyz=-0.0313 0 0 rpy=0 0 0
- added joint j_dg_3_1: type revolute, parent l_dg_base, child l_dg_3_1, origin xyz=-0.013279 -0.023 0.0712 rpy=0 0 0, axis 0 0 1, limit lower=-1.5707963267948966 upper=2.129301687433082 effort=7.644 velocity=3.141592653589793
- added joint j_dg_3_2: type revolute, parent l_dg_3_1, child l_dg_3_2, origin xyz=0 0 0.0405 rpy=0 0 0, axis -1 0 0, limit lower=-1.5707963267948966 upper=1.5707963267948966 effort=7.644 velocity=3.141592653589793
- added joint j_dg_3_3: type revolute, parent l_dg_3_2, child l_dg_3_3, origin xyz=-0.0242 0 0.029 rpy=0 0 0, axis 0 1 0, limit lower=-0.0 upper=2.8099800957108707 effort=7.644 velocity=3.141592653589793
- added joint j_dg_3_4: type revolute, parent l_dg_3_3, child l_dg_3_4, origin xyz=-0.0434 0 0 rpy=0 0 0, axis 0 1 0, limit lower=-1.5707963267948966 upper=1.8675022996339325 effort=7.644 velocity=3.141592653589793
- added joint j_dg_3_tip: type fixed, parent l_dg_3_4, child l_dg_3_tip, origin xyz=-0.0313 0 0 rpy=0 0 0
- added joint j_dg_dg_base: type fixed, parent l_dg_mount, child l_dg_base, origin xyz=0 0 0.004 rpy=0 0 0
