Commit message: update dg3fm model.

File: dg_description/urdf/dg3f_m.xacro (robot description, xacro)
@@ -1,29 +1,35 @@
 <?xml version="1.0" ?>
-<!-- Please note that the physical values of the URDF are not yet complete and will be modified in the future. -->
 <!--
-    dg3f_m.xacro
-Please note that the physical values of the URDF are not yet complete and will be modified in the future.
+    dg3f_m.urdf
     Licensed under the BSD-3-Clause
-    Copyright (c) 2025 Tesollo Inc.
+    Copyright (c) 2019-2025 Tesollo Inc.
     See LICENSE file for details.
     Reference:
     * https://tesollo.com/dg-3f/
 -->
-<robot name="dg3f_m" xmlns:xacro="http://www.ros.org/wiki/xacro">
-  <link name="base_link" />
-  <joint name="dummy_joint" type="fixed">
-    <origin xyz="0 0 0" rpy="0 0 0" />
-    <parent link="base_link" />
-  <child link="l_dg_base" />
-  </joint>
+<robot name="dg3f_m">
+  <link name="l_dg_mount">
+    <inertial>
+      <mass value="0.035" />
+    </inertial>
+    <visual>
+      <geometry>
+        <mesh filename="$(find dg_description)/meshes/dg3f_m/visual/l_dg_mount.dae"/>
+      </geometry>
+    </visual>
+    <collision>
+      <geometry>
+        <mesh filename="$(find dg_description)/meshes/dg3f_m/collision/l_dg_mount_c.STL"/>
+      </geometry>
+    </collision>
+  </link>
   <link name="l_dg_base">
     <inertial>
-      <origin xyz="-0.0022497 0.010893 0.10153" rpy="0.0 0.0 0.0" />
+      <origin xyz="0.00043337 0.00027389 0.044909" rpy="0 0 0" />
       <mass value="0.451" />
-      <inertia ixx="0.00058791" ixy="1.5175E-06" ixz="2.9558E-06" iyy="0.00059695" iyz="2.2019E-06"
-        izz="0.00047118" />
-    </inertial>
-    <visual>
-      <origin xyz="0.0 0.0 0.0" rpy="0.0 0.0 0.0" />
+      <inertia ixx="0.00074905" ixy="1.3406E-06" ixz="6.2559E-06" iyy="0.00076541" iyz="3.8906E-06" izz="0.00042544" />
+    </inertial>
+    <visual>
+      <origin xyz="0 0 0" rpy="0 0 0" />
       <geometry>
         <mesh filename="$(find dg_description)/meshes/dg3f_m/visual/l_dg_base.dae" />
@@ -31,5 +37,5 @@
     </visual>
     <collision>
-      <origin xyz="0.0 0.0 0.0" rpy="0.0 0.0 0.0" />
+      <origin xyz="0 0 0" rpy="0 0 0" />
       <geometry>
         <mesh filename="$(find dg_description)/meshes/dg3f_m/collision/l_dg_base_c.STL" />
@@ -37,135 +43,135 @@
     </collision>
   </link>
-  <!--finger1-->
-  <link name="l_dg_1_1">
-    <inertial>
-      <origin xyz="0.022193 0.00068612 0.031323" rpy="0.0 0.0 0.0" />
-      <mass value="0.046" />
-      <inertia ixx="1.2546E-05" ixy="2.0811E-12" ixz="2.9703E-06" iyy="1.4339E-05" iyz="-4.5421E-12"
-        izz="4.4982E-06" />
-    </inertial>
-    <visual>
-      <origin xyz="0.0 0.0 0.0" rpy="0.0 0.0 0.0" />
-      <geometry>
-        <mesh filename="$(find dg_description)/meshes/dg3f_m/visual/l_dg_1_1.dae" />
-      </geometry>
-    </visual>
-    <collision>
-      <origin xyz="0.0 0.0 0.0" rpy="0.0 0.0 0.0" />
-      <geometry>
-        <mesh filename="$(find dg_description)/meshes/dg3f_m/collision/l_dg_1_1_c.STL" />
+  <joint name="j_dg_dg_base" type="fixed">
+    <parent link="l_dg_mount"/>
+    <child link="l_dg_base"/>
+    <origin rpy="0 0 0" xyz="0 0 0.004"/>
+  </joint>
+<!--finger1-->
+<link name="l_dg_1_1">
+    <inertial>
+      <origin xyz="0.0039774 -8.829E-09 0.020057" rpy="0 0 0" />
+      <mass value="0.0493" />
+      <inertia ixx="1.3247E-05" ixy="1.7768E-12" ixz="2.91E-06" iyy="1.5031E-05" iyz="-6.8008E-12" izz="4.5216E-06" />
+    </inertial>
+    <visual>
+      <origin xyz="0 0 0" rpy="0 0 0" />
+      <geometry>
+        <mesh filename="$(find dg_description)/meshes/dg3f_m/visual/l_1_1.dae" />
+      </geometry>
+    </visual>
+    <collision>
+      <origin xyz="0 0 0" rpy="0 0 0" />
+      <geometry>
+        <mesh filename="$(find dg_description)/meshes/dg3f_m/collision/l_1_1_c.STL" />
       </geometry>
     </collision>
   </link>
   <joint name="j_dg_1_1" type="revolute">
-    <origin xyz="0.02656 0.0 0.0807" rpy="0.0 0.0 0.0" />
+    <origin xyz="0.026558 0 0.0712" rpy="0 0 0" />
     <parent link="l_dg_base" />
     <child link="l_dg_1_1" />
     <axis xyz="0 0 1" />
-    <limit lower="-1.5708" upper="1.5708" effort="7.644" velocity="3.141592653589793" />
+    <limit lower="-1.5707963267948966" upper="1.5707963267948966" effort="7.644" velocity="3.141592653589793" />
   </joint>
   <link name="l_dg_1_2">
     <inertial>
-      <origin xyz="0.0024353 0.0097149 -0.01236" rpy="0.0 0.0 0.0" />
-      <mass value="0.027" />
-      <inertia ixx="2.2017E-06" ixy="-7.2176E-08" ixz="-7.7488E-07" iyy="5.9914E-06"
-        iyz="-9.3255E-08" izz="5.8581E-06" />
-    </inertial>
-    <visual>
-      <origin xyz="0.0 0.0 0.0" rpy="0.0 0.0 0.0" />
-      <geometry>
-        <mesh filename="$(find dg_description)/meshes/dg3f_m/visual/l_dg_1_2.dae" />
-      </geometry>
-    </visual>
-    <collision>
-      <origin xyz="0.0 0.0 0.0" rpy="0.0 0.0 0.0" />
-      <geometry>
-        <mesh filename="$(find dg_description)/meshes/dg3f_m/collision/l_dg_1_2_c.STL" />
+      <origin xyz="0.013085 -0.00032847 0.013274" rpy="0 0 0" />
+      <mass value="0.0191" />
+      <inertia ixx="2.4921E-06" ixy="1.1229E-07" ixz="-1.0064E-06" iyy="6.5468E-06" iyz="1.5916E-07" izz="6.2269E-06" />
+    </inertial>
+    <visual>
+      <origin xyz="0 0 0" rpy="0 0 0" />
+      <geometry>
+        <mesh filename="$(find dg_description)/meshes/dg3f_m/visual/l_1_2.dae" />
+      </geometry>
+    </visual>
+    <collision>
+      <origin xyz="0 0 0" rpy="0 0 0" />
+      <geometry>
+        <mesh filename="$(find dg_description)/meshes/dg3f_m/collision/l_1_2_c.STL" />
       </geometry>
     </collision>
   </link>
   <joint name="j_dg_1_2" type="revolute">
-    <origin xyz="0.0005 0.0 0.04" rpy="0.0 0.0 0.0" />
+    <origin xyz="0 0 0.0405" rpy="0 0 0" />
     <parent link="l_dg_1_1" />
     <child link="l_dg_1_2" />
     <axis xyz="1 0 0" />
-    <limit lower="-1.76278" upper="1.76278" effort="7.644" velocity="3.141592653589793" />
+    <limit lower="-1.5707963267948966" upper="1.5707963267948966" effort="7.644" velocity="3.141592653589793" />
   </joint>
   <link name="l_dg_1_3">
     <inertial>
-      <origin xyz="-0.14886 0.032543 0.99997" rpy="0.0 0.0 0.0" />
-      <mass value="0.045" />
-      <inertia ixx="2.6509E-06" ixy="-3.4446E-07" ixz="2.2529E-08" iyy="6.9707E-06" iyz="4.0639E-09"
-        izz="7.6E-06" />
-    </inertial>
-    <visual>
-      <origin xyz="0.0 0.0 0.0" rpy="0.0 0.0 0.0" />
-      <geometry>
-        <mesh filename="$(find dg_description)/meshes/dg3f_m/visual/l_dg_1_3.dae" />
-      </geometry>
-    </visual>
-    <collision>
-      <origin xyz="0.0 0.0 0.0" rpy="0.0 0.0 0.0" />
-      <geometry>
-        <mesh filename="$(find dg_description)/meshes/dg3f_m/collision/l_dg_1_3_c.STL" />
+      <origin xyz="0.015926 -0.0001838 -1.5688E-05" rpy="0 0 0" />
+      <mass value="0.04535" />
+      <inertia ixx="2.7201E-06" ixy="5.68E-07" ixz="1.3288E-08" iyy="7.7224E-06" iyz="-3.8255E-11" izz="8.3935E-06" />
+    </inertial>
+    <visual>
+      <origin xyz="0 0 0" rpy="0 0 0" />
+      <geometry>
+        <mesh filename="$(find dg_description)/meshes/dg3f_m/visual/l_1_3.dae" />
+      </geometry>
+    </visual>
+    <collision>
+      <origin xyz="0 0 0" rpy="0 0 0" />
+      <geometry>
+        <mesh filename="$(find dg_description)/meshes/dg3f_m/collision/l_1_3_c.STL" />
       </geometry>
     </collision>
   </link>
   <joint name="j_dg_1_3" type="revolute">
-    <origin xyz="0.0237 0.0 0.029" rpy="0.0 0.0 0.0" />
+    <origin xyz="0.0242 0 0.029" rpy="0 0 0" />
     <parent link="l_dg_1_2" />
     <child link="l_dg_1_3" />
     <axis xyz="0 -1 0" />
-    <limit lower="-0.15708" upper="2.53073" effort="7.644" velocity="3.141592653589793" />
+    <limit lower="-0.0" upper="2.8099800957108707" effort="7.644" velocity="3.141592653589793" />
   </joint>
   <link name="l_dg_1_4">
     <inertial>
-      <origin xyz="-0.030524 -0.0005434 0.027713" rpy="0.0 0.0 0.0" />
-      <mass value="0.041" />
-      <inertia ixx="2.2664E-06" ixy="-5.9942E-08" ixz="4.2521E-09" iyy="3.4239E-06"
-        iyz="-5.8003E-12" izz="3.6584E-06" />
-    </inertial>
-    <visual>
-      <origin xyz="0.0 0.0 0.0" rpy="0.0 0.0 0.0" />
-      <geometry>
-        <mesh filename="$(find dg_description)/meshes/dg3f_m/visual/l_dg_1_4.dae" />
-      </geometry>
-    </visual>
-    <collision>
-      <origin xyz="0.0 0.0 0.0" rpy="0.0 0.0 0.0" />
-      <geometry>
-        <mesh filename="$(find dg_description)/meshes/dg3f_m/collision/l_dg_1_4_c.STL" />
+      <origin xyz="0.013887 0.00026201 -4.6519E-10" rpy="0 0 0" />
+      <mass value="0.0408" />
+      <inertia ixx="2.3785E-06" ixy="7.7437E-08" ixz="-4.9155E-14" iyy="3.5656E-06" iyz="1.1628E-12" izz="3.8056E-06" />
+    </inertial>
+    <visual>
+      <origin xyz="0 0 0" rpy="0 0 0" />
+      <geometry>
+        <mesh filename="$(find dg_description)/meshes/dg3f_m/visual/l_1_4.dae" />
+      </geometry>
+    </visual>
+    <collision>
+      <origin xyz="0 0 0" rpy="0 0 0" />
+      <geometry>
+        <mesh filename="$(find dg_description)/meshes/dg3f_m/collision/l_1_4_c.STL" />
       </geometry>
     </collision>
   </link>
   <joint name="j_dg_1_4" type="revolute">
-    <origin xyz="0.0434 0.0 0.0" rpy="0.0 0.0 0.0" />
+    <origin xyz="0.0434 0 0" rpy="0 0 0" />
     <parent link="l_dg_1_3" />
     <child link="l_dg_1_4" />
     <axis xyz="0 -1 0" />
-    <limit lower="-0.226893" upper="2.02458" effort="7.644" velocity="3.141592653589793" />
+    <limit lower="-1.5707963267948966" upper="1.8675022996339325" effort="7.644" velocity="3.141592653589793" />
   </joint>
   <link name="l_dg_1_tip">
     <inertial>
-      <origin xyz="-0.001569 0.010965 0.0099767" rpy="0.0 0.0 0.0" />
-      <mass value="0.015" />
-      <inertia ixx="8.959E-07" ixy="-9.5229E-11" ixz="6.4892E-08" iyy="8.7791E-07" iyz="-1.3588E-11"
-        izz="1.04E-06" />
-    </inertial>
-    <visual>
-      <origin xyz="0.0 0.0 0.0" rpy="0.0 0.0 0.0" />
-      <geometry>
-        <mesh filename="$(find dg_description)/meshes/dg3f_m/visual/l_dg_1_tip.dae" />
-      </geometry>
-    </visual>
-    <collision>
-      <origin xyz="0.0 0.0 0.0" rpy="0.0 0.0 0.0" />
-      <geometry>
-        <mesh filename="$(find dg_description)/meshes/dg3f_m/collision/l_dg_1_tip_c.STL" />
+      <origin xyz="0.010984 -8.1442E-09 -0.00048894" rpy="0 0 0" />
+      <mass value="0.0172" />
+      <inertia ixx="1.1855E-06" ixy="5.5892E-12" ixz="9.3654E-08" iyy="1.439E-06" iyz="-1.6025E-11" izz="1.6355E-06" />
+    </inertial>
+    <visual>
+      <origin xyz="0 0 0" rpy="0 0 0" />
+      <geometry>
+        <mesh filename="$(find dg_description)/meshes/dg3f_m/visual/l_1_tip.dae" />
+      </geometry>
+    </visual>
+    <collision>
+      <origin xyz="0 0 0" rpy="0 0 0" />
+      <geometry>
+        <mesh filename="$(find dg_description)/meshes/dg3f_m/collision/l_1_tip_c.STL" />
       </geometry>
     </collision>
   </link>
   <joint name="j_dg_1_tip" type="fixed">
-    <origin xyz="0.0298 0.0 0.0" rpy="0.0 0.0 0.0" />
+    <origin xyz="0.0313 0 0" rpy="0 0 0" />
     <parent link="l_dg_1_4" />
     <child link="l_dg_1_tip" />
@@ -174,132 +180,127 @@
   <link name="l_dg_2_1">
     <inertial>
-      <origin xyz="0.022193 0.00068612 0.031323" rpy="0.0 0.0 0.0" />
-      <mass value="0.046" />
-      <inertia ixx="1.2546E-05" ixy="2.0811E-12" ixz="2.9703E-06" iyy="1.4339E-05" iyz="-4.5421E-12"
-        izz="4.4982E-06" />
-    </inertial>
-    <visual>
-      <origin xyz="0.0 0.0 0.0" rpy="0.0 0.0 0.0" />
-      <geometry>
-        <mesh filename="$(find dg_description)/meshes/dg3f_m/visual/l_dg_2_1.dae" />
-      </geometry>
-    </visual>
-    <collision>
-      <origin xyz="0.0 0.0 0.0" rpy="0.0 0.0 0.0" />
-      <geometry>
-        <mesh filename="$(find dg_description)/meshes/dg3f_m/collision/l_dg_2_1_c.STL" />
+      <origin xyz="-0.0039774 8.829E-09 0.020057" rpy="0 0 0" />
+      <mass value="0.0493" />
+      <inertia ixx="1.3247E-05" ixy="1.7768E-12" ixz="-2.91E-06" iyy="1.5031E-05" iyz="6.8008E-12" izz="4.5216E-06" />
+    </inertial>
+    <visual>
+      <origin xyz="0 0 0" rpy="0 0 0" />
+      <geometry>
+        <mesh filename="$(find dg_description)/meshes/dg3f_m/visual/l_23_1.dae" />
+      </geometry>
+    </visual>
+    <collision>
+      <origin xyz="0 0 0" rpy="0 0 0" />
+      <geometry>
+        <mesh filename="$(find dg_description)/meshes/dg3f_m/collision/l_23_1_c.STL" />
       </geometry>
     </collision>
   </link>
   <joint name="j_dg_2_1" type="revolute">
-    <origin xyz="-0.01328 0.023 0.0807" rpy="0.0 0.0 0.0" />
+    <origin xyz="-0.013279 0.023 0.0712" rpy="0 0 0" />
     <parent link="l_dg_base" />
     <child link="l_dg_2_1" />
     <axis xyz="0 0 1" />
-    <limit lower="-1.5708" upper="0.5236" effort="7.644" velocity="3.141592653589793" />
+    <limit lower="-2.129301687433082" upper="1.5707963267948966" effort="7.644" velocity="3.141592653589793" />
   </joint>
   <link name="l_dg_2_2">
     <inertial>
-      <origin xyz="0.0024353 0.0097149 -0.01236" rpy="0.0 0.0 0.0" />
-      <mass value="0.027" />
-      <inertia ixx="2.2017E-06" ixy="-7.2176E-08" ixz="-7.7488E-07" iyy="5.9914E-06"
-        iyz="-9.3255E-08" izz="5.8581E-06" />
-    </inertial>
-    <visual>
-      <origin xyz="0.0 0.0 0.0" rpy="0.0 0.0 0.0" />
-      <geometry>
-        <mesh filename="$(find dg_description)/meshes/dg3f_m/visual/l_dg_2_2.dae" />
-      </geometry>
-    </visual>
-    <collision>
-      <origin xyz="0.0 0.0 0.0" rpy="0.0 0.0 0.0" />
-      <geometry>
-        <mesh filename="$(find dg_description)/meshes/dg3f_m/collision/l_dg_2_2_c.STL" />
+      <origin xyz="-0.013085 0.00032847 0.013274" rpy="0 0 0" />
+      <mass value="0.0191" />
+      <inertia ixx="2.4921E-06" ixy="1.1229E-07" ixz="1.0064E-06" iyy="6.5468E-06" iyz="-1.5916E-07" izz="6.2269E-06" />
+    </inertial>
+    <visual>
+      <origin xyz="0 0 0" rpy="0 0 0" />
+      <geometry>
+        <mesh filename="$(find dg_description)/meshes/dg3f_m/visual/l_23_2.dae" />
+      </geometry>
+    </visual>
+    <collision>
+      <origin xyz="0 0 0" rpy="0 0 0" />
+      <geometry>
+        <mesh filename="$(find dg_description)/meshes/dg3f_m/collision/l_23_2_c.STL" />
       </geometry>
     </collision>
   </link>
   <joint name="j_dg_2_2" type="revolute">
-    <origin xyz="-0.0005 0.0 0.04" rpy="0.0 0.0 0.0" />
+    <origin xyz="0 0 0.0405" rpy="0 0 0" />
     <parent link="l_dg_2_1" />
     <child link="l_dg_2_2" />
     <axis xyz="-1 0 0" />
-    <limit lower="-1.76278" upper="1.76278" effort="7.644" velocity="3.141592653589793" />
+    <limit lower="-1.5707963267948966" upper="1.5707963267948966" effort="7.644" velocity="3.141592653589793" />
   </joint>
   <link name="l_dg_2_3">
     <inertial>
-      <origin xyz="-0.14886 0.032543 0.99997" rpy="0.0 0.0 0.0" />
-      <mass value="0.045" />
-      <inertia ixx="2.6509E-06" ixy="-3.4446E-07" ixz="2.2529E-08" iyy="6.9707E-06" iyz="4.0639E-09"
-        izz="7.6E-06" />
-    </inertial>
-    <visual>
-      <origin xyz="0.0 0.0 0.0" rpy="0.0 0.0 0.0" />
-      <geometry>
-        <mesh filename="$(find dg_description)/meshes/dg3f_m/visual/l_dg_2_3.dae" />
-      </geometry>
-    </visual>
-    <collision>
-      <origin xyz="0.0 0.0 0.0" rpy="0.0 0.0 0.0" />
-      <geometry>
-        <mesh filename="$(find dg_description)/meshes/dg3f_m/collision/l_dg_2_3_c.STL" />
+      <origin xyz="-0.0159258962872331 0.000183796044363631 -1.56883420763254E-05" rpy="0 0 0" />
+      <mass value="0.04535" />
+      <inertia ixx="2.72014634088682E-06" ixy="5.67998480575708E-07" ixz="-1.32884157040829E-08" iyy="7.72244376203872E-06" iyz="3.82553595666275E-11" izz="8.39345564298784E-06" />
+    </inertial>
+    <visual>
+      <origin xyz="0 0 0" rpy="0 0 0" />
+      <geometry>
+        <mesh filename="$(find dg_description)/meshes/dg3f_m/visual/l_23_3.dae" />
+      </geometry>
+    </visual>
+    <collision>
+      <origin xyz="0 0 0" rpy="0 0 0" />
+      <geometry>
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
File: dg_description/urdf/dg5f_left.urdf (robot description, URDF)
Before this commit: robot dg5f_left, 28 links, 27 joints
Links:
- link ll_dg_1_1: geometry collision mesh filename=package://dg_description/meshes/dg5f_left/collision/ll_dg_1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; visual mesh filename=package://dg_description/meshes/dg5f_left/visual/ll_dg_1_1.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
- link ll_dg_1_2: geometry collision mesh filename=package://dg_description/meshes/dg5f_left/collision/ll_dg_1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; visual mesh filename=package://dg_description/meshes/dg5f_left/visual/ll_dg_1_2.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
- link ll_dg_1_3: geometry collision mesh filename=package://dg_description/meshes/dg5f_left/collision/ll_dg_1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; visual mesh filename=package://dg_description/meshes/dg5f_left/visual/ll_dg_1_3.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
- link ll_dg_1_4: geometry collision mesh filename=package://dg_description/meshes/dg5f_left/collision/ll_dg_1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; visual mesh filename=package://dg_description/meshes/dg5f_left/visual/ll_dg_1_4.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
- link ll_dg_1_tip: geometry collision mesh filename=package://dg_description/meshes/dg5f_left/collision/ll_dg_1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; visual mesh filename=package://dg_description/meshes/dg5f_left/visual/ll_dg_1_ti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
- link ll_dg_2_1: geometry collision mesh filename=package://dg_description/meshes/dg5f_left/collision/ll_dg_2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; visual mesh filename=package://dg_description/meshes/dg5f_left/visual/ll_dg_2_1.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
- link ll_dg_2_2: geometry collision mesh filename=package://dg_description/meshes/dg5f_left/collision/ll_dg_2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; visual mesh filename=package://dg_description/meshes/dg5f_left/visual/ll_dg_2_2.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
- link ll_dg_2_3: geometry collision mesh filename=package://dg_description/meshes/dg5f_left/collision/ll_dg_2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; visual mesh filename=package://dg_description/meshes/dg5f_left/visual/ll_dg_2_3.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
- link ll_dg_2_4: geometry collision mesh filename=package://dg_description/meshes/dg5f_left/collision/ll_dg_2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; visual mesh filename=package://dg_description/meshes/dg5f_left/visual/ll_dg_2_4.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
- link ll_dg_2_tip: geometry collision mesh filename=package://dg_description/meshes/dg5f_left/collision/ll_dg_2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; visual mesh filename=package://dg_description/meshes/dg5f_left/visual/ll_dg_2_ti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
- link ll_dg_3_1: geometry collision mesh filename=package://dg_description/meshes/dg5f_left/collision/ll_dg_3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; visual mesh filename=package://dg_description/meshes/dg5f_left/visual/ll_dg_3_1.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
- link ll_dg_3_2: geometry collision mesh filename=package://dg_description/meshes/dg5f_left/collision/ll_dg_3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; visual mesh filename=package://dg_description/meshes/dg5f_left/visual/ll_dg_3_2.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
- link ll_dg_3_3: geometry collision mesh filename=package://dg_description/meshes/dg5f_left/collision/ll_dg_3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; visual mesh filename=package://dg_description/meshes/dg5f_left/visual/ll_dg_3_3.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
- link ll_dg_3_4: geometry collision mesh filename=package://dg_description/meshes/dg5f_left/collision/ll_dg_3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; visual mesh filename=package://dg_description/meshes/dg5f_left/visual/ll_dg_3_4.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
- link ll_dg_3_tip: geometry collision mesh filename=package://dg_description/meshes/dg5f_left/collision/ll_dg_3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; visual mesh filename=package://dg_description/meshes/dg5f_left/visual/ll_dg_3_ti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
- link ll_dg_4_1: geometry collision mesh filename=package://dg_description/meshes/dg5f_left/collision/ll_dg_4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; visual mesh filename=package://dg_description/meshes/dg5f_left/visual/ll_dg_4_1.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
- link ll_dg_4_2: geometry collision mesh filename=package://dg_description/meshes/dg5f_left/collision/ll_dg_4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; visual mesh filename=package://dg_description/meshes/dg5f_left/visual/ll_dg_4_2.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
- link ll_dg_4_3: geometry collision mesh filename=package://dg_description/meshes/dg5f_left/collision/ll_dg_4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; visual mesh filename=package://dg_description/meshes/dg5f_left/visual/ll_dg_4_3.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
- link ll_dg_4_4: geometry collision mesh filename=package://dg_description/meshes/dg5f_left/collision/ll_dg_4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; visual mesh filename=package://dg_description/meshes/dg5f_left/visual/ll_dg_4_4.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
- link ll_dg_4_tip: geometry collision mesh filename=package://dg_description/meshes/dg5f_left/collision/ll_dg_4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; visual mesh filename=package://dg_description/meshes/dg5f_left/visual/ll_dg_4_ti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
- link ll_dg_5_1: geometry collision mesh filename=package://dg_description/meshes/dg5f_left/collision/ll_dg_5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; visual mesh filename=package://dg_description/meshes/dg5f_left/visual/ll_dg_5_1.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
- link ll_dg_5_2: geometry collision mesh filename=package://dg_description/meshes/dg5f_left/collision/ll_dg_5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; visual mesh filename=package://dg_description/meshes/dg5f_left/visual/ll_dg_5_2.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
- link ll_dg_5_3: geometry collision mesh filename=package://dg_description/meshes/dg5f_left/collision/ll_dg_5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; visual mesh filename=package://dg_description/meshes/dg5f_left/visual/ll_dg_5_3.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
- link ll_dg_5_4: geometry collision mesh filename=package://dg_description/meshes/dg5f_left/collision/ll_dg_5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; visual mesh filename=package://dg_description/meshes/dg5f_left/visual/ll_dg_5_4.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
- link ll_dg_5_tip: geometry collision mesh filename=package://dg_description/meshes/dg5f_left/collision/ll_dg_5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; visual mesh filename=package://dg_description/meshes/dg5f_left/visual/ll_dg_5_ti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
- link ll_dg_base: geometry collision mesh filename=package://dg_description/meshes/dg5f_left/collision/ll_dg_b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; visual mesh filename=package://dg_description/meshes/dg5f_left/visual/ll_dg_base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
- link ll_dg_mount: geometry collision mesh filename=package://dg_description/meshes/dg5f_left/collision/ll_dg_m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; visual mesh filename=package://dg_description/meshes/dg5f_left/visual/ll_dg_moun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
- link ll_dg_palm: geometry collision mesh filename=package://dg_description/meshes/dg5f_left/collision/ll_dg_p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; visual mesh filename=package://dg_description/meshes/dg5f_left/visual/ll_dg_palm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

File: dg_description/urdf/dg5f_left.xacro (robot description, xacro)
@@ -10,5 +10,5 @@
 <robot name="dg5f_left" xmlns:xacro="http://www.ros.org/wiki/xacro">
   <link name="left_base_link" />
-  <joint name="base_joint" type="fixed">
+  <joint name="base_joint2" type="fixed">
     <origin xyz="0 0 0" rpy="0 0 0" />
     <parent link="left_base_link" />
