Commit message: update dg3fm model.

File: dg_description/urdf/dg5f_right.urdf (robot description, URDF)
Before this commit: robot dg5f_right, 28 links, 27 joints
Links:
- link rl_dg_1_1: geometry collision mesh filename=package://dg_description/meshes/dg5f_right/collision/rl_dg_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; visual mesh filename=package://dg_description/meshes/dg5f_right/visual/rl_dg_1_1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
- link rl_dg_1_2: geometry collision mesh filename=package://dg_description/meshes/dg5f_right/collision/rl_dg_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; visual mesh filename=package://dg_description/meshes/dg5f_right/visual/rl_dg_1_2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
- link rl_dg_1_3: geometry collision mesh filename=package://dg_description/meshes/dg5f_right/collision/rl_dg_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; visual mesh filename=package://dg_description/meshes/dg5f_right/visual/rl_dg_1_3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
- link rl_dg_1_4: geometry collision mesh filename=package://dg_description/meshes/dg5f_right/collision/rl_dg_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; visual mesh filename=package://dg_description/meshes/dg5f_right/visual/rl_dg_1_4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
- link rl_dg_1_tip: geometry collision mesh filename=package://dg_description/meshes/dg5f_right/collision/rl_dg_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; visual mesh filename=package://dg_description/meshes/dg5f_right/visual/rl_dg_1_t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
- link rl_dg_2_1: geometry collision mesh filename=package://dg_description/meshes/dg5f_right/collision/rl_dg_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; visual mesh filename=package://dg_description/meshes/dg5f_right/visual/rl_dg_2_1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
- link rl_dg_2_2: geometry collision mesh filename=package://dg_description/meshes/dg5f_right/collision/rl_dg_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; visual mesh filename=package://dg_description/meshes/dg5f_right/visual/rl_dg_2_2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
- link rl_dg_2_3: geometry collision mesh filename=package://dg_description/meshes/dg5f_right/collision/rl_dg_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; visual mesh filename=package://dg_description/meshes/dg5f_right/visual/rl_dg_2_3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
- link rl_dg_2_4: geometry collision mesh filename=package://dg_description/meshes/dg5f_right/collision/rl_dg_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; visual mesh filename=package://dg_description/meshes/dg5f_right/visual/rl_dg_2_4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
- link rl_dg_2_tip: geometry collision mesh filename=package://dg_description/meshes/dg5f_right/collision/rl_dg_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; visual mesh filename=package://dg_description/meshes/dg5f_right/visual/rl_dg_2_t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
- link rl_dg_3_1: geometry collision mesh filename=package://dg_description/meshes/dg5f_right/collision/rl_dg_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; visual mesh filename=package://dg_description/meshes/dg5f_right/visual/rl_dg_3_1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
- link rl_dg_3_2: geometry collision mesh filename=package://dg_description/meshes/dg5f_right/collision/rl_dg_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; visual mesh filename=package://dg_description/meshes/dg5f_right/visual/rl_dg_3_2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
- link rl_dg_3_3: geometry collision mesh filename=package://dg_description/meshes/dg5f_right/collision/rl_dg_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; visual mesh filename=package://dg_description/meshes/dg5f_right/visual/rl_dg_3_3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
- link rl_dg_3_4: geometry collision mesh filename=package://dg_description/meshes/dg5f_right/collision/rl_dg_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; visual mesh filename=package://dg_description/meshes/dg5f_right/visual/rl_dg_3_4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
- link rl_dg_3_tip: geometry collision mesh filename=package://dg_description/meshes/dg5f_right/collision/rl_dg_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; visual mesh filename=package://dg_description/meshes/dg5f_right/visual/rl_dg_3_t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
- link rl_dg_4_1: geometry collision mesh filename=package://dg_description/meshes/dg5f_right/collision/rl_dg_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; visual mesh filename=package://dg_description/meshes/dg5f_right/visual/rl_dg_4_1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
- link rl_dg_4_2: geometry collision mesh filename=package://dg_description/meshes/dg5f_right/collision/rl_dg_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; visual mesh filename=package://dg_description/meshes/dg5f_right/visual/rl_dg_4_2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
- link rl_dg_4_3: geometry collision mesh filename=package://dg_description/meshes/dg5f_right/collision/rl_dg_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; visual mesh filename=package://dg_description/meshes/dg5f_right/visual/rl_dg_4_3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
- link rl_dg_4_4: geometry collision mesh filename=package://dg_description/meshes/dg5f_right/collision/rl_dg_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; visual mesh filename=package://dg_description/meshes/dg5f_right/visual/rl_dg_4_4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
- link rl_dg_4_tip: geometry collision mesh filename=package://dg_description/meshes/dg5f_right/collision/rl_dg_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; visual mesh filename=package://dg_description/meshes/dg5f_right/visual/rl_dg_4_t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
- link rl_dg_5_1: geometry collision mesh filename=package://dg_description/meshes/dg5f_right/collision/rl_dg_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; visual mesh filename=package://dg_description/meshes/dg5f_right/visual/rl_dg_5_1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
- link rl_dg_5_2: geometry collision mesh filename=package://dg_description/meshes/dg5f_right/collision/rl_dg_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; visual mesh filename=package://dg_description/meshes/dg5f_right/visual/rl_dg_5_2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
- link rl_dg_5_3: geometry collision mesh filename=package://dg_description/meshes/dg5f_right/collision/rl_dg_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; visual mesh filename=package://dg_description/meshes/dg5f_right/visual/rl_dg_5_3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
- link rl_dg_5_4: geometry collision mesh filename=package://dg_description/meshes/dg5f_right/collision/rl_dg_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; visual mesh filename=package://dg_description/meshes/dg5f_right/visual/rl_dg_5_4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
- link rl_dg_5_tip: geometry collision mesh filename=package://dg_description/meshes/dg5f_right/collision/rl_dg_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; visual mesh filename=package://dg_description/meshes/dg5f_right/visual/rl_dg_5_t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
- link rl_dg_base: geometry collision mesh filename=package://dg_description/meshes/dg5f_right/collision/rl_dg_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; visual mesh filename=package://dg_description/meshes/dg5f_right/visual/rl_dg_bas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
- link rl_dg_mount: geometry collision mesh filename=package://dg_description/meshes/dg5f_right/collision/rl_dg_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; visual mesh filename=package://dg_description/meshes/dg5f_right/visual/rl_dg_mou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
- link rl_dg_palm: geometry collision mesh filename=package://dg_description/meshes/dg5f_right/collision/rl_dg_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; visual mesh filename=package://dg_description/meshes/dg5f_right/visual/rl_dg_pal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
