Commit message: Update dg3f_m.xacro

File: dg_description/urdf/dg3f_m.xacro (robot description, xacro)
@@ -9,4 +9,10 @@
 -->
 <robot name="dg3f_m">
+  <link name="base_link" />
+  <joint name="base_joint" type="fixed">
+    <origin xyz="0 0 0" rpy="0 0 0" />
+    <parent link="base_link" />
+    <child link="l_dg_mount" />
+  </joint>
   <link name="l_dg_mount">
     <inertial>
